Commit message: implement front only wheel

File: urdf/go2w_front_description.urdf (robot description, URDF)
Before this commit: robot go2w_description, 33 links, 32 joints
Links:
- removed link RL_foot_motor
- removed link RR_foot_motor
- added link RL_calf_rotor, mass 0.089
- added link RR_calf_rotor, mass 0.089
- added link RR_thigh_rotor, mass 0.089
- link RL_calf: geometry collision cylinder length=0.12 radius=0.013; visual mesh filename=./dae/calf1.dae
- link RL_foot: mass 0.520 -> 0.04; geometry collision sphere radius=0.022; visual mesh filename=./dae/foot.dae
- link RR_calf: geometry collision cylinder length=0.12 radius=0.013; visual mesh filename=./dae/calf_mirror1.dae
- link RR_foot: mass 0.520 -> 0.04; geometry collision sphere radius=0.022; visual mesh filename=./dae/foot.dae
Joints:
- removed joint RL_foot_motor_joint
- removed joint RR_foot_motor_joint
- added joint RL_calf_rotor_joint: type fixed, parent RL_thigh, child RL_calf_rotor, origin xyz=0 -0.03235 0 rpy=0 0 0
- added joint RR_calf_rotor_joint: type fixed, parent RR_thigh, child RR_calf_rotor, origin xyz=0 0.03235 0 rpy=0 0 0
- added joint RR_thigh_rotor_joint: type fixed, parent RR_hip, child RR_thigh_rotor, origin xyz=0 0.00015 0 rpy=0 0 0
- joint RL_foot_joint: axis 0 1 0 -> 0 0 0; limit effort=23.7 velocity=30.1 -> (none); origin xyz=0.0 0 -0.2264 rpy=0 0 0 -> xyz=0 0 -0.213 rpy=0 0 0; type continuous -> fixed
- joint RR_calf_joint: limit lower=-2.7227 upper=-0.83776 effort=35.55 velocity=20.07 -> lower=-2.7227 upper=-0.83776 effort=45.43 velocity=15.70
- joint RR_foot_joint: axis 0 1 0 -> 0 0 0; limit effort=23.7 velocity=30.1 -> (none); origin xyz=-0.0 0 -0.2264 rpy=0 0 0 -> xyz=0 0 -0.213 rpy=0 0 0; type continuous -> fixed
